File: stlink_adapter/sldrlss_stlink.kicad_pcb (KiCad board)
At the start: 2 copper layers, 17.8 x 17.8 mm, 2 parts, among them J1 Solderless, J2 STLINK

Commit message: fabrication files
Other:
- board text added: "JLCJLCJLCJLC"
Changed lines of the file:
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@@
     (pad_to_mask_clearance 0)
     (pcbplotparams
-      (layerselection 0x00010fc_ffffffff)
+      (layerselection 0x00010f0_ffffffff)
       (disableapertmacros false)
       (usegerberextensions false)
@@
       (outputformat 1)
       (mirror false)
-      (drillshape 1)
+      (drillshape 0)
       (scaleselection 1)
-      (outputdirectory "")
+      (outputdirectory "gerber/")
     )
   )
@@
   (gr_line (start 96.52 44.45) (end 96.52 57.15) (layer "Edge.Cuts") (width 0.1))
   (gr_arc (start 111.76 41.91) (mid 113.556051 42.653949) (end 114.3 44.45) (layer "Edge.Cuts") (width 0.1))
+  (gr_text "JLCJLCJLCJLC" (at 99.06 50.8 90) (layer "B.SilkS")
+    (effects (font (size 1 1) (thickness 0.2)) (justify mirror))
+  )
   (gr_text "Laurent\nFiack" (at 100.076 57.404) (layer "F.SilkS")
     (effects (font (size 1 1) (thickness 0.15)))
